Commit message: Feat: Sero_2 kann sich in gazebo bewegen

File: src/sero_1/urdf/sero_1.urdf (robot description, URDF)
Before this commit: robot onshape, 7 links, 6 joints
Links:
- link base: mass 35.087052395247894765 -> 35.08705239524790187
- link link_3: mass 17.046409404154790224 -> 17.046409404154786671
Joints:
- joint 1: limit effort=1 velocity=20 -> lower=-3.141592653589793116 upper=3.141592653589793116 effort=1 velocity=20; origin xyz=1.873501354054951662e-16 0.055665231986508974249 0.10499999999999998224 rpy=3.141592653589793116 -0 0 -> xyz=1.8041113859237242606e-16 0.055665231986508988127 0.10499999999999999611 rpy=-3.1415926535897926719 6.8688042396975808885e-17 8.1606641769779487982e-06
- joint 2: limit effort=1 velocity=20 -> lower=-1.8110811019912356201 upper=1.8362307380071132279 effort=1 velocity=20; origin xyz=-6.9388939039073269853e-18 -0.059999999999999248379 -0.14500000000000001776 rpy=-1.57079632679489678 -2.2204460492503342815e-16 1.5707963267948943376 -> xyz=0 -0.060000000000000004718 -0.14500000000000001776 rpy=-1.570796326794896558 -0.46704913247174045798 1.570796326794896336
- joint 3: limit effort=1 velocity=20 -> lower=-3.2351423014966895764 upper=1.7570410727549981011 effort=1 velocity=20; origin xyz=-1.9428902930931246443e-17 0.44999999999999978906 8.0074835651082891598e-16 rpy=3.1415926535897864547 2.2759572004824394437e-15 -3.1415926535897926719 -> xyz=0 0.44999999999999995559 1.2533970036995509267e-18 rpy=3.141592653589793116 3.529925104387571233e-17 -2.8217730704100758565
- joint 4: limit effort=1 velocity=20 -> lower=-3.141592653589793116 upper=3.141592653589793116 effort=1 velocity=20; origin xyz=0.22000000000000724532 0.12083333333333379223 -0.016980779096483905599 rpy=3.1415926535897926719 1.570796326794891673 0 -> xyz=0.22000000000000002887 0.12083333333333334814 -0.016980779096484183155 rpy=-1.5707963268408067226 -1.5707952499523358814 1.5707963267450772982
- joint 5: limit effort=1 velocity=20 -> lower=-2.0653116879748694146 upper=2.0650581841370048153 effort=1 velocity=20; origin xyz=-0.030000000000000005829 -0.035000000000000031086 -0.18499999999999997002 rpy=-1.570796326794896558 1.8752360775309906313e-14 1.570796326794901665 -> xyz=-0.030000000000000016237 -0.035000000000000142109 -0.18499999999999999778 rpy=-1.570796326794896558 0.57407536946603265893 1.57079632679489678
- joint 6: limit effort=1 velocity=20 -> lower=-3.141592653589793116 upper=3.141592653589793116 effort=1 velocity=20; origin xyz=1.1102230246251565404e-16 0.080000000000000001665 -0.029500000000000005385 rpy=1.5707963267948958919 1.57079632679465786 0 -> xyz=1.1102230246251565404e-16 0.079999999999999960032 -0.029499999999999998446 rpy=1.5707963267948892305 -1.5707963265184670121 0

File: src/sero_2/urdf/sero_2.urdf (robot description, URDF)
Before this commit: robot onshape, 7 links, 6 joints
Links:
- added link world
- link base: mass 49.341703062128154045 -> 49.341703062128146939
- link link_01: mass 19.091905974861965944 -> 19.091905974861962392
- link link_02: mass 13.731956551120580556 -> 13.731956551120582333
- link link_05: mass 2.3102574452715733955 -> 2.3102574452715738396
Joints:
- removed joint 01
- removed joint 02
- removed joint 03
- removed joint 04
- removed joint 05
- added joint fixed_link_to_world: type fixed, parent world, child base
- added joint j1: type revolute, parent base, child link_01, origin xyz=-1.3877787807814459837e-17 0.060367606489668872161 0.12000000000000006495 rpy=-3.1415926535897793492 -8.8628477392845443571e-22 3.141592653589793116, axis 0 0 1, limit lower=-6.283185307 upper=6.283185307 effort=10 velocity=3.14
- added joint j2: type revolute, parent link_01, child link_02, origin xyz=-0.020000000000000003886 0.14873863542433760077 -0.20873863542433754303 rpy=1.5707963267948958919 0.855974613270912843 -1.57079632679489678, axis 0 0 1, limit lower=-1.8174 upper=0 effort=10 velocity=3.14
- added joint j3: type revolute, parent link_02, child link_03, origin xyz=0.47249999999999992006 5.5511151231257827021e-17 -0.039999999999999993894 rpy=-3.9099808047474802371e-16 6.5349778921725544513e-18 -1.8702914936790970835, axis 0 0 1, limit lower=0 upper=3.4906585039886590671 effort=10 velocity=3.14
- added joint j4: type revolute, parent link_03, child link_04, origin xyz=0.1052999999999999492 0 0.020000000000000059397 rpy=5.5511151231257814695e-17 -1.5707963267948952257 0, axis 0 0 1, limit lower=-6.283185307 upper=6.283185307 effort=10 velocity=3.14
- added joint j5: type revolute, parent link_04, child link_05, origin xyz=0.019999999999999986539 -1.1102230246251565404e-16 -0.32499999999999845679 rpy=1.5707963267948970021 -0.6422904971427879639 1.5707963267948992225, axis 0 0 1, limit lower=-1 upper=2.8792 effort=10 velocity=3.14
- joint fastened: limit effort=1 velocity=20 -> effort=10 velocity=3.14; origin xyz=-0.094999999999999862332 1.1102230246251565404e-16 -0.020000000000000003886 rpy=3.141592653589793116 -1.570796326794896558 0 -> xyz=-0.095000000000000028866 0 -0.019999999999999965722 rpy=3.141592653589793116 -1.5707963267948950037 0

File: src/sero_3/urdf/sero_3.urdf (robot description, URDF)
Before this commit: robot onshape, 10 links, 9 joints
Links:
- added link world
- link base: mass 100 -> 29.561020908170693389
- link ee_base: mass 13.798178184326978624 -> 13.798178184326982176
- link link_1: mass 32.098264787234512596 -> 32.098264787234505491
- link link_2: mass 95.41248128433817044 -> 95.412481284338156229
Joints:
- removed joint 1
- removed joint 2
- removed joint 3
- removed joint 4
- removed joint 5
- added joint fixed_link_to_world: type fixed, parent world, child base
- added joint j1: type revolute, parent base, child link_1, origin xyz=-4.1633363423443370266e-17 6.2524054036301313582e-17 0.17000000000000001221 rpy=3.141592653589793116 -3.5404820457539550914e-27 -5.5511151231290971505e-17, axis 0 0 1, limit lower=-3.141592653589793116 upper=3.141592653589793116 effort=320.98 velocity=2.95
- added joint j2: type revolute, parent link_1, child link_2, origin xyz=-6.1629758220391547298e-33 0.12000000000000005107 -0.079999999999999960032 rpy=1.5707963267948956698 -1.5707963267948956698 0, axis 0 0 1, limit lower=-1.5708 upper=1.5708 effort=954.12 velocity=4.37
- added joint j3: type revolute, parent link_2, child link_3, origin xyz=-0.62999999999999989342 -6.4711246131411124663e-32 1.061085658197035173e-17 rpy=-3.141592653589793116 -1.819226480685986761e-15 1.5707963267948961139, axis 0 0 1, limit lower=-3.141592653589793116 upper=3.141592653589793116 effort=2008.75 velocity=4.51
- added joint j4: type revolute, parent link_3, child link_4, origin xyz=-0.49500000000000005107 -0.14000000000000001332 -0.17000000000000009548 rpy=3.1415926535897917837 6.241086271459160841e-16 -3.1415926535897922278, axis 0 0 1, limit lower=-3.141592653589793116 upper=3.141592653589793116 effort=2008.75 velocity=3.32
- added joint j5: type revolute, parent link_4, child ee_base, origin xyz=0.14499999999999985123 -0.090000000000000301981 -0.079999999999999987788 rpy=-3.141592653589793116 1.5707963267948890085 0, axis 0 0 1, limit lower=-3.141592653589793116 upper=3.141592653589793116 effort=137.98 velocity=2.54
- joint vacuum_1: limit effort=1 velocity=20 -> effort=1 velocity=3.14; origin xyz=0.095000000000000014988 0.045000000000000039968 -0.035000000000000003331 rpy=1.1102230246251452005e-16 5.4470317145671831511e-16 1.570796326794896558 -> xyz=0.094999999999999987232 0.044999999999999706901 -0.035000000000000031086 rpy=-2.5673907444551896414e-16 -4.5080215706672108797e-30 1.570796326794896558
- joint vacuum_2: limit effort=1 velocity=20 -> effort=1 velocity=3.14; origin xyz=0.095000000000000028866 -0.044999999999999928946 -0.035000000000000031086 rpy=1.1102230246251452005e-16 5.4470317145671831511e-16 1.570796326794896558 -> xyz=0.095000000000000014988 -0.04500000000000015099 -0.035000000000000031086 rpy=-2.5673907444551896414e-16 -4.5080215706672108797e-30 1.570796326794896558
- joint vacuum_3: limit effort=1 velocity=20 -> effort=1 velocity=3.14; origin xyz=-0.09500000000000000111 0.045000000000000039968 -0.035000000000000031086 rpy=1.1102230246251452005e-16 5.4470317145671831511e-16 1.570796326794896558 -> xyz=-0.094999999999999987232 0.044999999999999706901 -0.035000000000000031086 rpy=-2.5673907444551896414e-16 -4.5080215706672108797e-30 1.570796326794896558
- joint vacuum_4: limit effort=1 velocity=20 -> effort=1 velocity=3.14; origin xyz=-0.094999999999999987232 -0.044999999999999928946 -0.035000000000000003331 rpy=1.1102230246251452005e-16 5.4470317145671831511e-16 1.570796326794896558 -> xyz=-0.094999999999999959477 -0.045000000000000373035 -0.035000000000000031086 rpy=-2.5673907444551896414e-16 -4.5080215706672108797e-30 1.570796326794896558

Commit message: Feat: Sero_1_moveit funktioniert. PID Regler ausbaufähig, aber funktional.

File: src/sero_1/urdf/sero_1.urdf (robot description, URDF)
Before this commit: robot onshape, 7 links, 6 joints
Links:
- added link world
Joints:
- removed joint 1
- removed joint 2
- removed joint 3
- removed joint 4
- removed joint 5
- removed joint 6
- added joint fixed_link_to_world: type fixed, parent world, child base
- added joint j1: type revolute, parent base, child link_1, origin xyz=1.8041113859237242606e-16 0.055665231986508988127 0.10499999999999999611 rpy=-3.1415926535897926719 6.8688042396975808885e-17 8.1606641769779487982e-06, axis 0 0 1, limit lower=-3.141592653589793116 upper=3.141592653589793116 effort=1000 velocity=1.18
- added joint j2: type revolute, parent link_1, child link_2, origin xyz=0 -0.060000000000000004718 -0.14500000000000001776 rpy=-1.570796326794896558 -0.46704913247174045798 1.570796326794896336, axis 0 0 1, limit lower=-1.4 upper=2 effort=9000 velocity=100
- added joint j3: type revolute, parent link_2, child link_3, origin xyz=0 0.44999999999999995559 1.2533970036995509267e-18 rpy=3.141592653589793116 3.529925104387571233e-17 -2.8217730704100758565, axis 0 0 1, limit lower=-1.35 upper=2.5 effort=1000 velocity=1.17
- added joint j4: type revolute, parent link_3, child link_4, origin xyz=0.22000000000000002887 0.12083333333333334814 -0.016980779096484183155 rpy=-1.5707963268408067226 -1.5707952499523358814 1.5707963267450772982, axis 0 0 1, limit lower=-3.141592653589793116 upper=3.141592653589793116 effort=1000 velocity=1.03
- added joint j5: type revolute, parent link_4, child link_5, origin xyz=-0.030000000000000016237 -0.035000000000000142109 -0.18499999999999999778 rpy=-1.570796326794896558 0.57407536946603265893 1.57079632679489678, axis 0 0 1, limit lower=-2.5 upper=1.7 effort=1000 velocity=1.01
- added joint jendeffector: type revolute, parent link_5, child endeffector, origin xyz=1.1102230246251565404e-16 0.079999999999999960032 -0.029499999999999998446 rpy=1.5707963267948892305 -1.5707963265184670121 0, axis 0 0 1, limit lower=-3.141592653589793116 upper=3.141592653589793116 effort=1000 velocity=1.02
