Commit message: Add workobject and link_attacher as submodule

File: src/sero_3/urdf/sero_3.urdf (robot description, URDF)
Before this commit: robot onshape, 1 links, 0 joints
Links:
- added link ee_base, mass 13.798178184326978624; collision mesh filename=package://sero_3/meshes/ee_base.stl; visual mesh filename=package://sero_3/meshes/ee_base.stl
- added link link_1, mass 32.098264787234512596; collision mesh filename=package://sero_3/meshes/link_1.stl; visual mesh filename=package://sero_3/meshes/link_1.stl
- added link link_2, mass 95.41248128433817044; collision mesh filename=package://sero_3/meshes/link_2.stl; visual mesh filename=package://sero_3/meshes/link_2.stl
- added link link_3, mass 84.06211694702932391; collision mesh filename=package://sero_3/meshes/link_3.stl; visual mesh filename=package://sero_3/meshes/link_3.stl
- added link link_4, mass 35.563010627334307401; collision mesh filename=package://sero_3/meshes/link_4.stl; visual mesh filename=package://sero_3/meshes/link_4.stl
- added link v_tube, mass 0.16852026592631189073; collision mesh filename=package://sero_3/meshes/v_tube.stl; visual mesh filename=package://sero_3/meshes/v_tube.stl
- added link v_tube_2, mass 0.16852026592631189073; collision mesh filename=package://sero_3/meshes/v_tube.stl; visual mesh filename=package://sero_3/meshes/v_tube.stl
- added link v_tube_3, mass 0.16852026592631189073; collision mesh filename=package://sero_3/meshes/v_tube.stl; visual mesh filename=package://sero_3/meshes/v_tube.stl
- added link v_tube_4, mass 0.16852026592631189073; collision mesh filename=package://sero_3/meshes/v_tube.stl; visual mesh filename=package://sero_3/meshes/v_tube.stl
- link base: mass 290.39841297718282931 -> 100; geometry collision mesh filename=package://sero_3/meshes/base.stl; visual mesh filename=package://sero_3/meshes/base.stl
Joints:
- added joint 1: type revolute, parent base, child link_1, origin xyz=2.2204460492503128343e-16 5.1067049100322390549e-17 0.14000000000000001332 rpy=3.141592653589793116 -2.0214560696288431017e-30 -5.5511151231257974933e-17, axis 0 0 1, limit effort=1 velocity=20
- added joint 2: type revolute, parent link_1, child link_2, origin xyz=8.5179240925324843315e-17 0.12000000000000103639 -0.080000000000000015543 rpy=1.570796326794896336 -0.71279526940051185502 -3.9647758287278457964e-16, axis 0 0 1, limit effort=1 velocity=20
- added joint 3: type revolute, parent link_2, child link_3, origin xyz=-0.6299999999999997824 1.3877787807814456755e-16 9.653611640754696961e-18 rpy=3.141592653589793116 -4.4594939066526483123e-16 2.428797384189281594, axis 0 0 1, limit effort=1 velocity=20
- added joint 4: type revolute, parent link_3, child link_4, origin xyz=-0.49499999999999999556 -0.1399999999999999023 -0.17000000000000009548 rpy=3.141592653589793116 6.548689762148525404e-18 3.141592653589793116, axis 0 0 1, limit effort=1 velocity=20
- added joint 5: type revolute, parent link_4, child ee_base, origin xyz=0.14499999999999990674 -0.090000000000000190958 -0.079999999999999987788 rpy=3.1415926535897926719 1.5707963267948952257 0, axis 0 0 1, limit effort=1 velocity=20
- added joint vacuum_1: type fixed, parent ee_base, child v_tube, origin xyz=0.095000000000000014988 0.045000000000000039968 -0.035000000000000003331 rpy=1.1102230246251452005e-16 5.4470317145671831511e-16 1.570796326794896558, axis 0 0 1, limit effort=1 velocity=20
- added joint vacuum_2: type fixed, parent ee_base, child v_tube_2, origin xyz=0.095000000000000028866 -0.044999999999999928946 -0.035000000000000031086 rpy=1.1102230246251452005e-16 5.4470317145671831511e-16 1.570796326794896558, axis 0 0 1, limit effort=1 velocity=20
- added joint vacuum_3: type fixed, parent ee_base, child v_tube_3, origin xyz=-0.09500000000000000111 0.045000000000000039968 -0.035000000000000031086 rpy=1.1102230246251452005e-16 5.4470317145671831511e-16 1.570796326794896558, axis 0 0 1, limit effort=1 velocity=20
- added joint vacuum_4: type fixed, parent ee_base, child v_tube_4, origin xyz=-0.094999999999999987232 -0.044999999999999928946 -0.035000000000000003331 rpy=1.1102230246251452005e-16 5.4470317145671831511e-16 1.570796326794896558, axis 0 0 1, limit effort=1 velocity=20

Commit message: Feat: Sero_3 kann sich nun auch in rviz und gazebo bewegen

File: src/sero_3/urdf/sero_3.urdf (robot description, URDF)
Before this commit: robot onshape, 11 links, 10 joints
Links:
- link ee_base: mass 13.798178184326982176 -> 5
- link link_1: mass 32.098264787234505491 -> 20
- link link_2: mass 95.412481284338156229 -> 10
- link link_3: mass 84.06211694702932391 -> 5
- link link_4: mass 35.563010627334307401 -> 10
Joints:
- joint j1: limit lower=-3.141592653589793116 upper=3.141592653589793116 effort=320.98 velocity=2.95 -> lower=-3.141592653589793116 upper=3.141592653589793116 effort=100 velocity=3.14
- joint j2: limit lower=-1.5708 upper=1.5708 effort=954.12 velocity=4.37 -> lower=-1.5708 upper=1.5708 effort=9000 velocity=3.14
- joint j3: limit lower=-3.141592653589793116 upper=3.141592653589793116 effort=2008.75 velocity=4.51 -> lower=-3.141592653589793116 upper=3.141592653589793116 effort=1000 velocity=3.14
- joint j4: limit lower=-3.141592653589793116 upper=3.141592653589793116 effort=2008.75 velocity=3.32 -> lower=-3.141592653589793116 upper=3.141592653589793116 effort=1000 velocity=3.14
- joint j5: limit lower=-3.141592653589793116 upper=3.141592653589793116 effort=137.98 velocity=2.54 -> lower=-3.141592653589793116 upper=3.141592653589793116 effort=1000 velocity=3.14
