Commit message: random update

File: src/3_R/urdf/urdf/3_R.urdf (robot description, URDF)
Before this commit: robot 3_robots, 21 links, 20 joints
Links:
- removed link base2
- removed link base3
- removed link link_1_3
- removed link link_2_3
- removed link link_3_3
- removed link link_4_3
- link base: mass 35.08705239524790187 -> 29.561020908170693389; geometry collision mesh filename=package://sero_3/meshes/base.stl; visual mesh filename=package://sero_3/meshes/base.stl
- link link_1: mass 18.368766956758115327 -> 20; geometry collision mesh filename=package://sero_3/meshes/link_1.stl; visual mesh filename=package://sero_3/meshes/link_1.stl
- link link_2: mass 23.673948033547031145 -> 10; geometry collision mesh filename=package://sero_3/meshes/link_2.stl; visual mesh filename=package://sero_3/meshes/link_2.stl
- link link_3: mass 17.046409404154786671 -> 5; geometry collision mesh filename=package://sero_3/meshes/link_3.stl; visual mesh filename=package://sero_3/meshes/link_3.stl
- link link_4: mass 3.4104383191089318039 -> 10; geometry collision mesh filename=package://sero_3/meshes/link_4.stl; visual mesh filename=package://sero_3/meshes/link_4.stl
Joints:
- joint fixed_link_to_world_2: child base2 -> base
- joint fixed_link_to_world_3: child base3 -> base
- joint j1_2: parent base2 -> base
- joint j1_3: child link_1_3 -> link_1; parent base3 -> base
- joint j2_3: child link_2_3 -> link_2; parent link_1_3 -> link_1
- joint j3_3: child link_3_3 -> link_3; parent link_2_3 -> link_2
- joint j4_3: child link_4_3 -> link_4; parent link_3_3 -> link_3
- joint j5_3: parent link_4_3 -> link_4
