Commit message: corrected urdf

File: src/multirobot/urdf/multirobot_backup.urdf (robot description, URDF)
Before this commit: robot multirobot, 25 links, 24 joints
Joints:
- removed joint fastened
- added joint sero_2_j6: type fixed, parent sero_2_link_5, child sero_2_endeffector, origin xyz=-0.095000000000000028866 0 -0.019999999999999965722 rpy=3.141592653589793116 -1.5707963267948950037 0, axis 0 0 1, limit effort=1 velocity=20
- joint sero_2_j2: limit lower=0.54105206811824213542 upper=2.3212879051524581975 effort=1 velocity=20 -> lower=-1.8174 upper=0 effort=1 velocity=20
