Commit message: added friction and damping to multirobot_moveit configuration

File: src/multirobot/urdf/multirobot.urdf (robot description, URDF)
Before this commit: robot multirobot, 25 links, 24 joints
Joints:
- joint sero_1_j1: limit lower=-3.141592653589793116 upper=3.141592653589793116 effort=1 velocity=20 -> lower=-3.141592653589793116 upper=3.141592653589793116 effort=1000 velocity=20
- joint sero_1_j2: limit lower=-1.8110811019912356201 upper=1.8362307380071132279 effort=1 velocity=20 -> lower=-1.8110811019912356201 upper=1.8362307380071132279 effort=1000 velocity=20
- joint sero_1_j3: limit lower=-3.2351423014966895764 upper=1.7570410727549981011 effort=1 velocity=20 -> lower=-3.2351423014966895764 upper=1.7570410727549981011 effort=1000 velocity=20
- joint sero_1_j4: limit lower=-3.141592653589793116 upper=3.141592653589793116 effort=1 velocity=20 -> lower=-3.141592653589793116 upper=3.141592653589793116 effort=1000 velocity=20
- joint sero_1_j5: limit lower=-2.0653116879748694146 upper=2.0650581841370048153 effort=1 velocity=20 -> lower=-2.0653116879748694146 upper=2.0650581841370048153 effort=1000 velocity=20
- joint sero_1_j6: limit lower=-3.141592653589793116 upper=3.141592653589793116 effort=1 velocity=20 -> lower=-3.141592653589793116 upper=3.141592653589793116 effort=1000 velocity=20
- joint sero_2_j1: limit lower=-3.141592653589793116 upper=3.141592653589793116 effort=1 velocity=20 -> lower=-3.141592653589793116 upper=3.141592653589793116 effort=1000 velocity=20
- joint sero_2_j2: limit lower=-1.8174 upper=0 effort=1 velocity=20 -> lower=-1.8174 upper=0 effort=1000 velocity=20
- joint sero_2_j3: limit lower=-0.36651914291880921537 upper=3.4906585039886590671 effort=1 velocity=20 -> lower=-0.36651914291880921537 upper=3.4906585039886590671 effort=1000 velocity=20
- joint sero_2_j4: limit lower=-3.141592653589793116 upper=3.141592653589793116 effort=1 velocity=20 -> lower=-3.141592653589793116 upper=3.141592653589793116 effort=1000 velocity=20
- joint sero_2_j5: limit lower=-0.1570796326794896558 upper=3.2812189937493396741 effort=1 velocity=20 -> lower=-0.1570796326794896558 upper=3.2812189937493396741 effort=1000 velocity=20
- joint sero_2_j6: limit effort=1 velocity=20 -> effort=1000 velocity=20
- joint sero_3_j1: limit lower=-3.141592653589793116 upper=3.141592653589793116 effort=1 velocity=20 -> lower=-3.141592653589793116 upper=3.141592653589793116 effort=1000 velocity=20
- joint sero_3_j2: limit lower=0 upper=3.141592653589793116 effort=1 velocity=20 -> lower=0 upper=3.141592653589793116 effort=1000 velocity=20
- joint sero_3_j3: limit lower=-3.141592653589793116 upper=3.141592653589793116 effort=1 velocity=20 -> lower=-3.141592653589793116 upper=3.141592653589793116 effort=1000 velocity=20
- joint sero_3_j4: limit lower=-3.141592653589793116 upper=3.141592653589793116 effort=1 velocity=20 -> lower=-3.141592653589793116 upper=3.141592653589793116 effort=1000 velocity=20
- joint sero_3_j5: limit lower=-3.141592653589793116 upper=3.141592653589793116 effort=1 velocity=20 -> lower=-3.141592653589793116 upper=3.141592653589793116 effort=1000 velocity=20
- joint sero_3_vacuum_1: limit effort=1 velocity=20 -> effort=1000 velocity=20
- joint sero_3_vacuum_2: limit effort=1 velocity=20 -> effort=1000 velocity=20
- joint sero_3_vacuum_3: limit effort=1 velocity=20 -> effort=1000 velocity=20
- joint sero_3_vacuum_4: limit effort=1 velocity=20 -> effort=1000 velocity=20

Commit message: A few changes for better functionality. Simulation does not work cleanly yet

File: src/multirobot/urdf/multirobot.urdf (robot description, URDF)
Before this commit: robot multirobot, 25 links, 24 joints
Links:
- link sero_3_base: mass 29.561020908170693389 -> 9.853673636
- link sero_3_endeffector_base: mass 13.798178184326982176 -> 4.5993927281089940587
- link sero_3_link_1: mass 32.098264787234505491 -> 10.699421596
- link sero_3_link_2: mass 95.412481284338156229 -> 31.804160428
- link sero_3_link_3: mass 84.06211694702932391 -> 28.02070564900977464
- link sero_3_link_4: mass 35.563010627334307401 -> 11.854336875778102467
- link sero_3_v_tube: mass 0.16852026592631189073 -> 0.05617342197543729691
- link sero_3_v_tube_2: mass 0.16852026592631189073 -> 0.05617342197543729691
- link sero_3_v_tube_3: mass 0.16852026592631189073 -> 0.05617342197543729691
- link sero_3_v_tube_4: mass 0.16852026592631189073 -> 0.05617342197543729691
Joints:
- removed joint fixed_link_to_world
- removed joint sero_1_to_sero_2
- removed joint sero_2_to_sero_3
- added joint fixed_link_to_world_sero_1: type fixed, parent world, child sero_1_base, origin xyz=0 0 0 rpy=0 0 0
- added joint fixed_link_to_world_sero_2: type fixed, parent world, child sero_2_base, origin xyz=1 0 0 rpy=0 0 0
- added joint fixed_link_to_world_sero_3: type fixed, parent world, child sero_3_base, origin xyz=0 1 0 rpy=0 0 0
- joint sero_1_j1: limit lower=-3.141592653589793116 upper=3.141592653589793116 effort=1000 velocity=20 -> lower=-3.141592653589793116 upper=3.141592653589793116 effort=100000 velocity=200
- joint sero_1_j2: limit lower=-1.8110811019912356201 upper=1.8362307380071132279 effort=1000 velocity=20 -> lower=-1.8110811019912356201 upper=1.8362307380071132279 effort=100000 velocity=200
- joint sero_1_j3: limit lower=-3.2351423014966895764 upper=1.7570410727549981011 effort=1000 velocity=20 -> lower=-3.2351423014966895764 upper=1.7570410727549981011 effort=100000 velocity=200
- joint sero_1_j4: limit lower=-3.141592653589793116 upper=3.141592653589793116 effort=1000 velocity=20 -> lower=-3.141592653589793116 upper=3.141592653589793116 effort=100000 velocity=200
- joint sero_1_j5: limit lower=-2.0653116879748694146 upper=2.0650581841370048153 effort=1000 velocity=20 -> lower=-2.0653116879748694146 upper=2.0650581841370048153 effort=100000 velocity=200
- joint sero_1_j6: limit lower=-3.141592653589793116 upper=3.141592653589793116 effort=1000 velocity=20 -> lower=-3.141592653589793116 upper=3.141592653589793116 effort=100000 velocity=200
- joint sero_2_j1: limit lower=-3.141592653589793116 upper=3.141592653589793116 effort=1000 velocity=20 -> lower=-3.141592653589793116 upper=3.141592653589793116 effort=100000 velocity=200
- joint sero_2_j2: limit lower=-1.8174 upper=0 effort=1000 velocity=20 -> lower=-1.8174 upper=0 effort=100000 velocity=200
- joint sero_2_j3: limit lower=-0.36651914291880921537 upper=3.4906585039886590671 effort=1000 velocity=20 -> lower=-0.36651914291880921537 upper=3.4906585039886590671 effort=100000 velocity=200
- joint sero_2_j4: limit lower=-3.141592653589793116 upper=3.141592653589793116 effort=1000 velocity=20 -> lower=-3.141592653589793116 upper=3.141592653589793116 effort=100000 velocity=200
- joint sero_2_j5: limit lower=-0.1570796326794896558 upper=3.2812189937493396741 effort=1000 velocity=20 -> lower=-0.1570796326794896558 upper=3.2812189937493396741 effort=100000 velocity=200
- joint sero_2_j6: limit effort=1000 velocity=20 -> effort=100000 velocity=200
- joint sero_3_j1: limit lower=-3.141592653589793116 upper=3.141592653589793116 effort=1000 velocity=20 -> lower=-3.141592653589793116 upper=3.141592653589793116 effort=100000 velocity=200
- joint sero_3_j2: limit lower=0 upper=3.141592653589793116 effort=1000 velocity=20 -> lower=-1.5707963267948956698 upper=1.5707963267948956698 effort=100000 velocity=200
- joint sero_3_j3: limit lower=-3.141592653589793116 upper=3.141592653589793116 effort=1000 velocity=20 -> lower=-3.141592653589793116 upper=3.141592653589793116 effort=100000 velocity=200
- joint sero_3_j4: limit lower=-3.141592653589793116 upper=3.141592653589793116 effort=1000 velocity=20 -> lower=-3.141592653589793116 upper=3.141592653589793116 effort=100000 velocity=200
- joint sero_3_j5: limit lower=-3.141592653589793116 upper=3.141592653589793116 effort=1000 velocity=20 -> lower=-3.141592653589793116 upper=3.141592653589793116 effort=100000 velocity=200
- joint sero_3_vacuum_1: limit effort=1000 velocity=20 -> effort=100000 velocity=200
- joint sero_3_vacuum_2: limit effort=1000 velocity=20 -> effort=100000 velocity=200
- joint sero_3_vacuum_3: limit effort=1000 velocity=20 -> effort=100000 velocity=200
- joint sero_3_vacuum_4: limit effort=1000 velocity=20 -> effort=100000 velocity=200
