Commit message: stuck in urdf

File: src/3_robots/urdf/3_robots.urdf (robot description, URDF)
Before this commit: robot 3_robots, 21 links, 20 joints
Links:
- link base3: geometry collision mesh filename=package://3_robots/meshes/base3.stl; visual mesh filename=package://3_robots/meshes/base3.stl
- link link_1_3: geometry collision mesh filename=package://3_robots/meshes/link_1_3.stl; visual mesh filename=package://3_robots/meshes/link_1_3.stl
- link link_2_3: geometry collision mesh filename=package://3_robots/meshes/link_2_3.stl; visual mesh filename=package://3_robots/meshes/link_2_3.stl
- link link_3_3: geometry collision mesh filename=package://3_robots/meshes/link_3.stl; visual mesh filename=package://3_robots/meshes/link_3_3.stl
- link link_4_3: geometry collision mesh filename=package://3_robots/meshes/link_4_3.stl; visual mesh filename=package://3_robots/meshes/link_4_3.stl
- link v_tube: geometry collision mesh filename=package://3_robots/meshes/v_tube.stl; visual mesh filename=package://3_robots/meshes/v_tube.stl
