Commit message: Fix: Nils

File: src/sero_multi_station/robot_description/sero_multi_station.urdf (robot description, URDF)
Before this commit: robot sero_multi_station, 25 links, 24 joints
Links:
- link sero_3_base: mass 29.561020908170693389 -> 50
- link sero_3_endeffector_base: mass 13.798178184326982176 -> 2.759635637
- link sero_3_link_1: mass 32.098264787234505491 -> 6.419652957
- link sero_3_link_2: mass 95.412481284338156229 -> 19.082496257
- link sero_3_link_3: mass 84.06211694702932391 -> 16.812423389
- link sero_3_link_4: mass 35.563010627334307401 -> 7.112602125

Commit message: Added TCP and joints to planning groups

File: src/sero_multi_station/robot_description/sero_multi_station.urdf (robot description, URDF)
Before this commit: robot sero_multi_station, 25 links, 24 joints
Links:
- added link sero_1_tcp
- added link sero_2_tcp
- added link sero_3_tcp
Joints:
- added joint sero_1_jtcp: type fixed, parent sero_1_endeffector, child sero_1_tcp, origin xyz=0  -0.060828  -0.205 rpy=0 0 0
- added joint sero_2_jtcp: type fixed, parent sero_2_endeffector, child sero_2_tcp, origin xyz=0 0 -0.100 rpy=0 0 0
- added joint sero_3_jtcp: type fixed, parent sero_3_endeffector_base, child sero_3_tcp, origin xyz=0 0 -0.08 rpy=0 0 0
