Commit message: Changed workobject and its spawning

File: src/station_peripherals/urdf/workobject.urdf (robot description, URDF)
Before this commit: robot workobject, 1 links, 0 joints
Links:
- added link world
- link workobject_link: mass 0.2 -> 50.0; geometry collision mesh filename=package://station_peripherals/meshes/workobject.stl scale=0.001 0.001 0.001; visual mesh filename=package://station_peripherals/meshes/workobject.stl scale=0.001 0.001 0.001
Joints:
- added joint workobject_joint: type fixed, parent world, child workobject_link, origin xyz=0.0 0.0 0.0 rpy=0.0 0.0 0.0
